Commit message: update for new gazebo

File: description/depth_camera.xacro (robot description, xacro)
@@ -22,13 +22,12 @@
     <gazebo reference="camera_link">
         <material>Gazebo/Red</material>
-        <sensor name="camera" type="camera">
+        <sensor name="camera" type="depth">
             <pose> 0 0 0 0 0 0 </pose>
             <visualize>true</visualize>
             <update_rate>10</update_rate>
-            <gz_frame_id>camera_rgb_frame</gz_frame_id>
             <camera>
                 <horizontal_fov>1.089</horizontal_fov>  <!--this unit is radians -->
                 <image>
-                    <format>R8G8B8</format>
+                    <format>B8G8R8</format>
                     <width>640</width>
                     <height>480</height>
@@ -41,4 +40,6 @@
             <plugin name="camera_controller" filename="libgazebo_ros_camera.so">
                 <frame_name>camera_link_optical</frame_name>
+                <min_depth>0.1</min_depth>
+                <max_depth>100.0</max_depth>
             </plugin>
         </sensor>

File: description/gazebo_control.xacro (robot description, xacro)
@@ -4,18 +4,29 @@
         <plugin filename="gz-sim-diff-drive-system" name="gz::sim::systems::DiffDrive">
             <!-- Wheel Information -->
-            <left_joint>left_wheek_joint</left_joint>
+            <left_joint>left_wheel_joint</left_joint>
             <right_joint>right_wheel_joint</right_joint>
             <wheel_separation>0.35</wheel_separation>
             <wheel_diameter>0.1</wheel_diameter>
             <!-- Limits -->
-            <max_wheel_torque>200</max_wheel_torque>
-            <max_wheel_acceleration>10.0</max_wheel_acceleration>
+            <!-- <max_wheel_torque>200</max_wheel_torque> -->
+            <max_linear_acceleration>10</max_linear_acceleration>
             <!-- Output -->
+            <odom_topic>odom</odom_topic>
             <frame_id>odom</frame_id>
             <child_frame_id>base_footprint</child_frame_id>
-            <publish_odom>true</publish_odom>
+            <odom_publisher_frequency>30</odom_publisher_frequency>
+            <topic>cmd_vel</topic>
+            <tf_topic>/tf</tf_topic>
+            <!-- <publish_odom>true</publish_odom>
             <publish_odom_tf>true</publish_odom_tf>
-            <publish_wheel_tf>true</publish_wheel_tf>
+            <publish_wheel_tf>true</publish_wheel_tf> -->
         </plugin>
+        <!-- Joint state publisher -->
+         <plugin filename="gz-sim-joint-state-publisher-system"
+          name="gz::sim::systems::JointStatePublisher">
+            <topic>joint_states</topic> <!-- from <ros><remapping> -->
+            <joint_name>left_wheel_joint</joint_name>
+            <joint_name>right_wheel_joint</joint_name>
+         </plugin>
     </gazebo>
 </robot>

File: description/lidar.xacro (robot description, xacro)
@@ -11,5 +11,5 @@
                 <cylinder radius="0.05" length="0.04"/>
             </geometry>
-            <material name="red "/>
+            <material name="red"/>
         </visual>
         <collision>
@@ -24,8 +24,9 @@
     <gazebo reference="laser_frame">
         <material>Gazebo/Red</material>
-        <sensor name="laser" type="ray">
-            <pose> 0 0 0 0 0 0 </pose>
-            <visualize>false</visualize>  <!-- if want to use, to change flag "true"-->
+        <sensor name="gpu_lidar" type="gpu_lidar">
+            <pose relative_to='laser_frame'> 0 0 0 0 0 0 </pose>
+            <topic>lidar</topic>
             <update_rate>10</update_rate>
+            <visualize>true</visualize>  <!-- if want to use, to change flag "true"-->
             <ray>
                 <scan>
@@ -41,10 +42,6 @@
                 </range>
             </ray>
-            <plugin name="laser_controller" filename="libgazebo_ros_ray_sensor.so">
-                <ros>
-                    <argument>~/out:=scan</argument>
-                </ros>
-                <output_type>sensor_msgs/LaserScan</output_type>
-                <frame_name>laser_frame</frame_name>
+            <plugin name="gz::sim::systems::Sensors" filename="gz-sim-sensors-system">
+                <render_engine>ogre2</render_engine>
             </plugin>
         </sensor>

File: description/robot.urdf.xacro (robot description, xacro)
@@ -1,7 +1,14 @@
 <?xml version="1.0"?>
-<robot xmlns:xacro="http://www.ros.org/wiki/xacro"  name="robot">
+<robot xmlns:xacro="http://www.ros.org/wiki/xacro"  name="differential_drive_robot">
     <xacro:include filename="robot_core.xacro" />
-    <xacro:include filename="gazebo_control.xacro" />
+    <xacro:arg name="use_ros2_control" default="false"/>
+    <xacro:if value="$(arg use_ros2_control)">
+        <xacro:include filename="ros2_control.xacro" />
+    </xacro:if>
+    <xacro:unless value="$(arg use_ros2_control)">
+        <xacro:include filename="gazebo_control.xacro" />
+    </xacro:unless>
     <xacro:include filename="lidar.xacro" />
     <xacro:include filename="camera.xacro" />
+    <!-- <xacro:include filename="depth_camera.xacro" /> -->
 </robot>

File: description/robot_core.xacro (robot description, xacro)
@@ -60,4 +60,6 @@
         <origin xyz="0 0.175 0" rpy="-${pi/2} 0 0"/>
         <axis xyz="0 0 1"/>
+        <limit effort="200" velocity="10"/>
+        <dynamics damping="1.0" friction="1.0"/>
     </joint>
     <link name="left_wheel">
@@ -77,5 +79,7 @@
         </xacro:inertial_cylinder>
     </link>
-    <gazebo reference="lef_wheel">
+    <gazebo reference="left_wheel">
+        <mu1>0.2</mu1>
+        <mu2>0.2</mu2>
         <material>Gazebo/Blue</material>
     </gazebo>
@@ -86,4 +90,6 @@
         <origin xyz="0 -0.175 0" rpy="${pi/2} 0 0"/>
         <axis xyz="0 0 -1"/>
+        <limit effort="200" velocity="10"/>
+        <dynamics damping="1.0" friction="1.0"/>
     </joint>
     <link name="right_wheel">
@@ -104,4 +110,6 @@
     </link>
     <gazebo reference="right_wheel">
+        <mu1>0.2</mu1>
+        <mu2>0.2</mu2>
         <material>Gazebo/Blue</material>
     </gazebo>
