Commit message: added base_footprint link

File: description/robot_core.xacro (robot description, xacro)
@@ -14,5 +14,12 @@
         <color rgba="0 0 0 1" />
     </material>
+    <!-- BASE FOOTPRINT -->
+    <link name="base_footprint"/>
     <!-- BASE LINK -->
+    <joint name="base_joint" type="fixed">
+        <parent link="base_footprint"/>
+        <child link="base_link"/>
+        <origin xyz="0 0 0.05" rpy="0 0 0"/>
+    </joint>
     <link name="base_link">
     </link>
@@ -41,4 +48,7 @@
         </xacro:inertial_box>
     </link>
+    <gazebo reference="chassis">
+        <material>Gazebo/White</material>
+    </gazebo>
     <!-- LEFT WHEEL LINK -->
     <joint name="left_wheel_joint" type="continuous">
@@ -64,4 +74,7 @@
         </xacro:inertial_cylinder>
     </link>
+    <gazebo reference="lef_wheel">
+        <material>Gazebo/Blue</material>
+    </gazebo>
     <!-- RIGHT WHEEL LINK -->
     <joint name="right_wheel_joint" type="continuous">
@@ -87,4 +100,7 @@
         </xacro:inertial_cylinder>
     </link>
+    <gazebo reference="right_wheel">
+        <material>Gazebo/Blue</material>
+    </gazebo>
     <!-- CASTER WHEEL LINK -->
     <joint name="caster_wheel_joint" type="fixed">
@@ -109,3 +125,6 @@
         </xacro:inertial_sphere>
     </link>
+    <gazebo reference="caster_wheel">
+        <material>Gazebo/Black</material>
+    </gazebo>
 </robot>

Commit message: updated robot_core file

File: description/robot_core.xacro (robot description, xacro)
@@ -60,5 +60,5 @@
         <origin xyz="0 0.175 0" rpy="-${pi/2} 0 0"/>
         <axis xyz="0 0 1"/>
-        <limit effort="2000" velocity="10"/>
+        <limit effort="2000" velocity="100"/>
         <dynamics damping="1.0" friction="1.0"/>
     </joint>
@@ -90,5 +90,5 @@
         <origin xyz="0 -0.175 0" rpy="${pi/2} 0 0"/>
         <axis xyz="0 0 -1"/>
-        <limit effort="2000" velocity="10"/>
+        <limit effort="2000" velocity="100"/>
         <dynamics damping="1.0" friction="1.0"/>
     </joint>

Commit message: updated robot_core file

File: description/robot_core.xacro (robot description, xacro)
@@ -60,5 +60,5 @@
         <origin xyz="0 0.175 0" rpy="-${pi/2} 0 0"/>
         <axis xyz="0 0 1"/>
-        <limit effort="2000" velocity="100"/>
+        <limit effort="2000" velocity="10"/>
         <dynamics damping="1.0" friction="1.0"/>
     </joint>
@@ -90,5 +90,5 @@
         <origin xyz="0 -0.175 0" rpy="${pi/2} 0 0"/>
         <axis xyz="0 0 -1"/>
-        <limit effort="2000" velocity="100"/>
+        <limit effort="2000" velocity="10"/>
         <dynamics damping="1.0" friction="1.0"/>
     </joint>
@@ -132,5 +132,5 @@
             </geometry>
         </collision>
-        <xacro:inertial_sphere mass="0.1" radius="0.035">
+        <xacro:inertial_sphere mass="0.05" radius="0.035">
             <origin xyz="0 0 0" rpy="0 0 0"/>
         </xacro:inertial_sphere>

Commit message: updated robot_core file

File: description/robot_core.xacro (robot description, xacro)
@@ -2,4 +2,21 @@
 <robot xmlns:xacro="http://www.ros.org/wiki/xacro">
     <xacro:include filename="inertial_macros.xacro"/>
+    <xacro:property name="chassis_length" value="0.22"/>
+    <xacro:property name="chassis_width" value="0.156"/>
+    <xacro:property name="chassis_height" value="0.082"/>
+    <xacro:property name="chassis_mass" value="1.0"/>
+    <xacro:property name="chassis_offset_z" value="0.008"/>
+    <xacro:property name="wheel_radius" value="0.033"/>
+    <xacro:property name="wheel_thickness" value="0.026"/>
+    <xacro:property name="wheel_mass" value="0.0385"/>
+    <xacro:property name="wheel_offset_x" value="0.06"/>
+    <xacro:property name="wheel_offset_y" value="0.093"/>
+    <xacro:property name="wheel_offset_z" value="0.033"/>
+    <xacro:property name="caster_wheel_radius" value="0.008"/>
+    <xacro:property name="caster_wheel_mass" value="0.02"/>
+    <xacro:property name="caster_wheel_offset_x" value="0.06"/>
+    <xacro:property name="caster_wheel_offset_z" value="0.008"/>
+    <xacro:property name="wheel_effort" value="2000"/>
+    <xacro:property name="wheel_velocity" value="30"/>
     <material name="white">
         <color rgba="1 1 1 1" />
@@ -23,5 +40,5 @@
         <parent link="base_footprint"/>
         <child link="base_link"/>
-        <origin xyz="0 0 0.008" rpy="0 0 0"/>
+        <origin xyz="0 0 ${chassis_offset_z}" rpy="0 0 0"/>
     </joint>
     <link name="base_link">
@@ -31,22 +48,22 @@
         <parent link="base_link"/>
         <child link="chassis"/>
-        <origin xyz="-0.06 0 0"/>
+        <origin xyz="${-wheel_offset_x} 0 0"/>
     </joint>
     <link name="chassis">
         <visual>
-            <origin xyz="0.11 0 0.041"/>
+            <origin xyz="${chassis_length/2} 0 ${chassis_height/2}"/>
             <geometry>
-                <box size="0.22 0.156 0.082"/>
+                <box size="${chassis_length} ${chassis_width} ${chassis_height}"/>
             </geometry>
             <material name="white"/>
         </visual>
         <collision>
-            <origin xyz="0.11 0 0.041"/>
+            <origin xyz="${chassis_length/2} 0 ${chassis_height/2}"/>
             <geometry>
-                <box size="0.22 0.156 0.082"/>
+                <box size="${chassis_length} ${chassis_width} ${chassis_height}"/>
             </geometry>
         </collision>
-        <xacro:inertial_box mass="1.0" x="0.22" y="0.156" z="0.082">
-            <origin xyz="0.11 0 0.041" rpy="0 0 0"/>
+        <xacro:inertial_box mass="${chassis_mass}" x="${chassis_length}" y="${chassis_width}" z="${chassis_height}">
+            <origin xyz="${chassis_length/2} 0 ${chassis_height/2}" rpy="0 0 0"/>
         </xacro:inertial_box>
     </link>
@@ -58,7 +75,7 @@
         <parent link="base_link"/>
         <child link="left_wheel"/>
-        <origin xyz="0 0.093 0.025" rpy="-${pi/2} 0 0"/>
+        <origin xyz="0 ${wheel_offset_y} ${wheel_offset_z - chassis_offset_z}" rpy="-${pi/2} 0 0"/>
         <axis xyz="0 0 1"/>
-        <limit effort="2000" velocity="30"/>
+        <limit effort="${wheel_effort}" velocity="${wheel_velocity}"/>
         <dynamics damping="1.0" friction="1.0"/>
     </joint>
@@ -66,5 +83,5 @@
         <visual>
             <geometry>
-                <cylinder radius="0.033" length="0.026"/>
+                <cylinder radius="${wheel_radius}" length="${wheel_thickness}"/>
             </geometry>
             <material name="blue"/>
@@ -72,8 +89,8 @@
         <collision>
             <geometry>
-                <cylinder radius="0.033" length="0.026"/>
+                <cylinder radius="${wheel_radius}" length="${wheel_thickness}"/>
             </geometry>
         </collision>
-        <xacro:inertial_cylinder mass="0.0385" length="0.026" radius="0.033">
+        <xacro:inertial_cylinder mass="${wheel_mass}" length="${wheel_thickness}" radius="${wheel_radius}">
             <origin xyz="0 0 0" rpy="0 0 0"/>
         </xacro:inertial_cylinder>
@@ -88,7 +105,7 @@
         <parent link="base_link"/>
         <child link="right_wheel"/>
-        <origin xyz="0 -0.093 0.025" rpy="${pi/2} 0 0"/>
+        <origin xyz="0 ${-wheel_offset_y} ${wheel_offset_z - chassis_offset_z}" rpy="${pi/2} 0 0"/>
         <axis xyz="0 0 -1"/>
-        <limit effort="2000" velocity="30"/>
+        <limit effort="${wheel_effort}" velocity="${wheel_velocity}"/>
         <dynamics damping="1.0" friction="1.0"/>
     </joint>
@@ -96,5 +113,5 @@
         <visual>
             <geometry>
-                <cylinder radius="0.033" length="0.026"/>
+                <cylinder radius="${wheel_radius}" length="${wheel_thickness}"/>
             </geometry>
             <material name="blue"/>
@@ -102,8 +119,8 @@
         <collision>
             <geometry>
-                <cylinder radius="0.033" length="0.026"/>
+                <cylinder radius="${wheel_radius}" length="${wheel_thickness}"/>
             </geometry>
         </collision>
-        <xacro:inertial_cylinder mass="0.0385" length="0.026" radius="0.033">
+        <xacro:inertial_cylinder mass="${wheel_mass}" length="${wheel_thickness}" radius="${wheel_radius}">
             <origin xyz="0 0 0" rpy="0 0 0"/>
         </xacro:inertial_cylinder>
@@ -118,10 +135,10 @@
         <parent link="chassis"/>
         <child link="caster_wheel"/>
-        <origin xyz="0.17 0 0"/>
+        <origin xyz="${chassis_length/2 + caster_wheel_offset_x} 0 0"/>
     </joint>
     <link name="caster_wheel">
         <visual>
             <geometry>
-                <sphere radius="0.008"/>
+                <sphere radius="${caster_wheel_radius}"/>
             </geometry>
             <material name="black"/>
@@ -129,8 +146,8 @@
         <collision>
             <geometry>
-                <sphere radius="0.008"/>
+                <sphere radius="${caster_wheel_radius}"/>
             </geometry>
         </collision>
-        <xacro:inertial_sphere mass="0.02" radius="0.008">
+        <xacro:inertial_sphere mass="${caster_wheel_mass}" radius="${caster_wheel_radius}">
             <origin xyz="0 0 0" rpy="0 0 0"/>
         </xacro:inertial_sphere>

Commit message: robot dimension change

File: description/robot_core.xacro (robot description, xacro)
@@ -3,18 +3,18 @@
     <xacro:include filename="inertial_macros.xacro"/>
     <xacro:property name="chassis_length" value="0.22"/>
-    <xacro:property name="chassis_width" value="0.156"/>
+    <xacro:property name="chassis_width" value="0.14"/>
     <xacro:property name="chassis_height" value="0.082"/>
     <xacro:property name="chassis_mass" value="1.0"/>
-    <xacro:property name="chassis_offset_z" value="0.008"/>
+    <xacro:property name="chassis_offset_z" value="0.015"/>
     <xacro:property name="wheel_radius" value="0.033"/>
     <xacro:property name="wheel_thickness" value="0.026"/>
     <xacro:property name="wheel_mass" value="0.0385"/>
-    <xacro:property name="wheel_offset_x" value="0.06"/>
-    <xacro:property name="wheel_offset_y" value="0.093"/>
+    <xacro:property name="wheel_offset_x" value="0.05"/>
+    <xacro:property name="wheel_offset_y" value="0.09"/>
     <xacro:property name="wheel_offset_z" value="0.033"/>
-    <xacro:property name="caster_wheel_radius" value="0.008"/>
+    <xacro:property name="caster_wheel_radius" value="0.015"/>
     <xacro:property name="caster_wheel_mass" value="0.02"/>
     <xacro:property name="caster_wheel_offset_x" value="0.06"/>
-    <xacro:property name="caster_wheel_offset_z" value="0.008"/>
+    <xacro:property name="caster_wheel_offset_z" value="0.015"/>
     <xacro:property name="wheel_effort" value="2000"/>
     <xacro:property name="wheel_velocity" value="30"/>
