Commit message: updated vehicle function

File: description/gazebo_control.xacro (robot description, xacro)
@@ -2,12 +2,13 @@
 <robot xmlns:xacro="http://www.ros.org/wiki/xacro">
     <gazebo>
-        <plugin name="gz::sim::systems::DiffDrive" filename="gz-sim-diff-drive-system">
+        <plugin filename="gz-sim-diff-drive-system" name="gz::sim::systems::DiffDrive">
             <!-- Wheel Information -->
             <left_joint>left_wheek_joint</left_joint>
             <right_joint>right_wheel_joint</right_joint>
-            <wheel_radius>0.05</wheel_radius>
+            <wheel_separation>0.35</wheel_separation>
+            <wheel_diameter>0.1</wheel_diameter>
             <!-- Limits -->
-            <max_effort>200</max_effort>
-            <max_linear_acceleration>10.0</max_linear_acceleration>
+            <max_wheel_torque>200</max_wheel_torque>
+            <max_wheel_acceleration>10.0</max_wheel_acceleration>
             <!-- Output -->
             <frame_id>odom</frame_id>

File: description/robot.urdf.xacro (robot description, xacro)
@@ -3,3 +3,5 @@
     <xacro:include filename="robot_core.xacro" />
     <xacro:include filename="gazebo_control.xacro" />
+    <xacro:include filename="lidar.xacro" />
+    <xacro:include filename="camera.xacro" />
 </robot>

File: description/robot_core.xacro (robot description, xacro)
@@ -13,4 +13,7 @@
     <material name="black">
         <color rgba="0 0 0 1" />
+    </material>
+    <material name="red">
+        <color rgba="1 0 0 1" />
     </material>
     <!-- BASE FOOTPRINT -->
@@ -127,4 +130,6 @@
     <gazebo reference="caster_wheel">
         <material>Gazebo/Black</material>
+        <mu1 value="0.001"/>
+        <mu2 value="0.001"/>
     </gazebo>
 </robot>

Commit message: update launch files

File: description/gazebo_control.xacro (robot description, xacro)
@@ -11,10 +11,10 @@
             <wheel_diameter>0.066</wheel_diameter>
             <!-- Limits -->
-            <max_linear_acceleration>10</max_linear_acceleration>
+            <max_linear_acceleration>30</max_linear_acceleration>
             <!-- Output -->
             <odom_topic>odom</odom_topic>
             <frame_id>odom</frame_id>
             <child_frame_id>base_footprint</child_frame_id>
-            <odom_publisher_frequency>30</odom_publisher_frequency>
+            <odom_publisher_frequency>5</odom_publisher_frequency>
             <topic>cmd_vel</topic>
             <tf_topic>tf</tf_topic>

File: description/robot.urdf.xacro (robot description, xacro)
@@ -2,5 +2,5 @@
 <robot xmlns:xacro="http://www.ros.org/wiki/xacro"  name="differential_drive_robot">
     <xacro:include filename="robot_core.xacro" />
-    <xacro:arg name="use_ros2_control" default="false"/>
+    <xacro:arg name="use_ros2_control" default="true"/>
     <xacro:if value="$(arg use_ros2_control)">
         <xacro:include filename="ros2_control.xacro" />

File: description/robot_core.xacro (robot description, xacro)
@@ -60,5 +60,5 @@
         <origin xyz="0 0.175 0" rpy="-${pi/2} 0 0"/>
         <axis xyz="0 0 1"/>
-        <limit effort="200" velocity="10"/>
+        <limit effort="2000" velocity="10"/>
         <dynamics damping="1.0" friction="1.0"/>
     </joint>
@@ -90,5 +90,5 @@
         <origin xyz="0 -0.175 0" rpy="${pi/2} 0 0"/>
         <axis xyz="0 0 -1"/>
-        <limit effort="200" velocity="10"/>
+        <limit effort="2000" velocity="10"/>
         <dynamics damping="1.0" friction="1.0"/>
     </joint>

Commit message: updated joystick yaml

File: description/gazebo_control.xacro (robot description, xacro)
@@ -13,4 +13,6 @@
             <max_linear_acceleration>10</max_linear_acceleration>
             <min_linear_acceleration>-10</min_linear_acceleration>
+            <max_linear_velocity>30</max_linear_velocity>
+            <min_linear_velocity>-30</min_linear_velocity>
             <!-- Output -->
             <odom_topic>odom</odom_topic>

File: description/robot_core.xacro (robot description, xacro)
@@ -60,5 +60,5 @@
         <origin xyz="0 0.175 0" rpy="-${pi/2} 0 0"/>
         <axis xyz="0 0 1"/>
-        <limit effort="2000" velocity="10"/>
+        <limit effort="2000" velocity="30"/>
         <dynamics damping="1.0" friction="1.0"/>
     </joint>
@@ -90,5 +90,5 @@
         <origin xyz="0 -0.175 0" rpy="${pi/2} 0 0"/>
         <axis xyz="0 0 -1"/>
-        <limit effort="2000" velocity="10"/>
+        <limit effort="2000" velocity="30"/>
         <dynamics damping="1.0" friction="1.0"/>
     </joint>

Commit message: updated gz_bridge.yaml

File: description/gazebo_control.xacro (robot description, xacro)
@@ -12,13 +12,14 @@
             <!-- Limits -->
             <max_linear_acceleration>10</max_linear_acceleration>
-            <min_linear_acceleration>-10</min_linear_acceleration>
-            <max_linear_velocity>30</max_linear_velocity>
-            <min_linear_velocity>-30</min_linear_velocity>
+            <!-- <min_linear_acceleration>-10</min_linear_acceleration> -->
+            <!-- <max_linear_velocity>30</max_linear_velocity>
+            <min_linear_velocity>-30</min_linear_velocity> -->
+            <!-- Input -->
+            <topic>cmd_vel</topic>
             <!-- Output -->
             <odom_topic>odom</odom_topic>
             <frame_id>odom</frame_id>
             <child_frame_id>base_footprint</child_frame_id>
-            <odom_publisher_frequency>5</odom_publisher_frequency>
-            <topic>cmd_vel</topic>
+            <odom_publish_frequency>5</odom_publish_frequency>
             <tf_topic>tf</tf_topic>
         </plugin>

File: description/robot_core.xacro (robot description, xacro)
@@ -69,5 +69,5 @@
     </link>
     <gazebo reference="chassis">
-        <material>Gazebo/White</material>
+        <material>Gazebo/Green</material>
     </gazebo>
     <!-- LEFT WHEEL LINK -->

File: description/ros2_control.xacro (robot description, xacro)
@@ -10,6 +10,6 @@
                 <param name="max">10</param>
             </command_interface>
+            <state_interface name="position"/>
             <state_interface name="velocity"/>
-            <state_interface name="position"/>
         </joint>
         <joint name="right_wheel_joint">
@@ -18,10 +18,10 @@
                 <param name="max">10</param>
             </command_interface>
+            <state_interface name="position"/>
             <state_interface name="velocity"/>
-            <state_interface name="position"/>
         </joint>
     </ros2_control>
     <gazebo>
-        <plugin filename="libgz_ros2_control-system.so" name="gz_ros2_control::GazeboSimROS2ControlPlugin">
+        <plugin filename="gz_ros2_control-system" name="gz_ros2_control::GazeboSimROS2ControlPlugin">
             <parameters>$(find vehicle_bot)/config/my_controllers.yaml</parameters>
             <controller_manager_prefix_node_name>controller_manager</controller_manager_prefix_node_name>
