Commit message: update gazebo_control

File: description/camera.xacro (robot description, xacro)
@@ -11,5 +11,5 @@
                 <box size="0.01 0.03 0.03"/>
             </geometry>
-            <material name="red "/>
+            <material name="red"/>
         </visual>
     </link>
@@ -20,13 +20,16 @@
     </joint>
     <link name="camera_link_optical"></link>
-    <gazebo reference="camera_link">
+    <gazebo reference="camera_link_optical">
         <material>Gazebo/Red</material>
-        <sensor name="camera" type="camera">
-            <pose> 0 0 0 0 0 0 </pose>
+        <sensor name="camera_link_optical" type="camera">
+            <pose> 0 0 0 ${pi/2} ${-pi/2} 0 </pose>
+            <always_on>true</always_on>
             <visualize>true</visualize>
             <update_rate>10</update_rate>
-            <gz_frame_id>camera_rgb_frame</gz_frame_id>
+            <topic>camera</topic>
+            <gz_frame_id>camera_link_optical</gz_frame_id>
             <camera>
-                <horizontal_fov>1.089</horizontal_fov>  <!--this unit is radians -->
+                <camera_info_topic>camera/camera_info</camera_info_topic>
+                <horizontal_fov>1.047</horizontal_fov>  <!-- this unit is radians -->
                 <image>
                     <format>R8G8B8</format>
@@ -39,7 +42,7 @@
                 </clip>
             </camera>
-            <plugin name="camera_controller" filename="libgazebo_ros_camera.so">
+            <!-- <plugin name="camera_controller" filename="libgazebo_ros_camera.so">
                 <frame_name>camera_link_optical</frame_name>
-            </plugin>
+            </plugin> -->
         </sensor>
     </gazebo>

File: description/depth_camera.xacro (robot description, xacro)
@@ -22,12 +22,15 @@
     <gazebo reference="camera_link">
         <material>Gazebo/Red</material>
-        <sensor name="camera" type="depth">
+        <sensor name="camera_link" type="depth">
             <pose> 0 0 0 0 0 0 </pose>
+            <always_on>true</always_on>
             <visualize>true</visualize>
             <update_rate>10</update_rate>
+            <topic>depth_camera/image_raw</topic>
+            <gz_frame_id>camera_link</gz_frame_id>
             <camera>
                 <horizontal_fov>1.089</horizontal_fov>  <!--this unit is radians -->
                 <image>
-                    <format>B8G8R8</format>
+                    <format>R_FLOAT32</format>
                     <width>640</width>
                     <height>480</height>
@@ -38,9 +41,9 @@
                 </clip>
             </camera>
-            <plugin name="camera_controller" filename="libgazebo_ros_camera.so">
+            <!-- <plugin name="camera_controller" filename="libgazebo_ros_camera.so">
                 <frame_name>camera_link_optical</frame_name>
                 <min_depth>0.1</min_depth>
                 <max_depth>100.0</max_depth>
-            </plugin>
+            </plugin> -->
         </sensor>
     </gazebo>

File: description/gazebo_control.xacro (robot description, xacro)
@@ -2,12 +2,13 @@
 <robot xmlns:xacro="http://www.ros.org/wiki/xacro">
     <gazebo>
+        <!-- Differential Drive -->
         <plugin filename="gz-sim-diff-drive-system" name="gz::sim::systems::DiffDrive">
             <!-- Wheel Information -->
             <left_joint>left_wheel_joint</left_joint>
             <right_joint>right_wheel_joint</right_joint>
+            <!-- Kinematics -->
             <wheel_separation>0.35</wheel_separation>
             <wheel_diameter>0.1</wheel_diameter>
             <!-- Limits -->
-            <!-- <max_wheel_torque>200</max_wheel_torque> -->
             <max_linear_acceleration>10</max_linear_acceleration>
             <!-- Output -->
@@ -18,15 +19,12 @@
             <topic>cmd_vel</topic>
             <tf_topic>/tf</tf_topic>
-            <!-- <publish_odom>true</publish_odom>
-            <publish_odom_tf>true</publish_odom_tf>
-            <publish_wheel_tf>true</publish_wheel_tf> -->
         </plugin>
         <!-- Joint state publisher -->
-         <plugin filename="gz-sim-joint-state-publisher-system"
+        <plugin filename="gz-sim-joint-state-publisher-system"
           name="gz::sim::systems::JointStatePublisher">
             <topic>joint_states</topic> <!-- from <ros><remapping> -->
             <joint_name>left_wheel_joint</joint_name>
             <joint_name>right_wheel_joint</joint_name>
-         </plugin>
+        </plugin>
     </gazebo>
 </robot>

File: description/lidar.xacro (robot description, xacro)
@@ -24,10 +24,12 @@
     <gazebo reference="laser_frame">
         <material>Gazebo/Red</material>
-        <sensor name="gpu_lidar" type="gpu_lidar">
-            <pose relative_to='laser_frame'> 0 0 0 0 0 0 </pose>
-            <topic>lidar</topic>
+        <sensor name="laser_frame" type="gpu_lidar">
+            <pose> 0 0 0 0 0 0 </pose>
+            <topic>scan</topic>
             <update_rate>10</update_rate>
+            <always_on>true</always_on>
             <visualize>true</visualize>  <!-- if want to use, to change flag "true"-->
-            <ray>
+            <gz_frame_id>laser_frame</gz_frame_id>
+            <lidar>
                 <scan>
                     <horizontal>
@@ -41,6 +43,6 @@
                     <max>12</max>
                 </range>
-            </ray>
-            <plugin name="gz::sim::systems::Sensors" filename="gz-sim-sensors-system">
+            </lidar>
+            <plugin filename="gz-sim-sensors-system" name="gz::sim::systems::Sensors">
                 <render_engine>ogre2</render_engine>
             </plugin>

File: description/robot.urdf.xacro (robot description, xacro)
@@ -2,5 +2,5 @@
 <robot xmlns:xacro="http://www.ros.org/wiki/xacro"  name="differential_drive_robot">
     <xacro:include filename="robot_core.xacro" />
-    <xacro:arg name="use_ros2_control" default="false"/>
+    <!-- <xacro:arg name="use_ros2_control" default="false"/>
     <xacro:if value="$(arg use_ros2_control)">
         <xacro:include filename="ros2_control.xacro" />
@@ -8,5 +8,6 @@
     <xacro:unless value="$(arg use_ros2_control)">
         <xacro:include filename="gazebo_control.xacro" />
-    </xacro:unless>
+    </xacro:unless> -->
+    <xacro:include filename="gazebo_control.xacro"/>
     <xacro:include filename="lidar.xacro" />
     <xacro:include filename="camera.xacro" />

File: description/robot_core.xacro (robot description, xacro)
@@ -60,5 +60,5 @@
         <origin xyz="0 0.175 0" rpy="-${pi/2} 0 0"/>
         <axis xyz="0 0 1"/>
-        <limit effort="200" velocity="10"/>
+        <limit effort="200" velocity="20"/>
         <dynamics damping="1.0" friction="1.0"/>
     </joint>
@@ -90,5 +90,5 @@
         <origin xyz="0 -0.175 0" rpy="${pi/2} 0 0"/>
         <axis xyz="0 0 -1"/>
-        <limit effort="200" velocity="10"/>
+        <limit effort="200" velocity="20"/>
         <dynamics damping="1.0" friction="1.0"/>
     </joint>

Commit message: update sdf file

File: description/camera.xacro (robot description, xacro)
@@ -22,4 +22,7 @@
     <gazebo reference="camera_link_optical">
         <material>Gazebo/Red</material>
+        <!-- <plugin filename="gz-sim-sensors-system" name="gz::sim::systems::Sensors">
+            <render_engine>ogre2</render_engine>
+        </plugin> -->
         <sensor name="camera_link_optical" type="camera">
             <pose> 0 0 0 ${pi/2} ${-pi/2} 0 </pose>
@@ -31,5 +34,5 @@
             <camera>
                 <camera_info_topic>camera/camera_info</camera_info_topic>
-                <horizontal_fov>1.047</horizontal_fov>  <!-- this unit is radians -->
+                <horizontal_fov>1.089</horizontal_fov>  <!-- this unit is radians -->
                 <image>
                     <format>R8G8B8</format>
@@ -42,11 +45,5 @@
                 </clip>
             </camera>
-            <!-- <plugin name="camera_controller" filename="libgazebo_ros_camera.so">
-                <frame_name>camera_link_optical</frame_name>
-            </plugin> -->
         </sensor>
-        <!-- <plugin filename="gz-sim-sensors-system" name="gz::sim::systems::Sensors">
-            <render_engine>ogre2</render_engine>
-        </plugin> -->
     </gazebo>
 </robot>

File: description/gazebo_control.xacro (robot description, xacro)
@@ -9,5 +9,5 @@
             <!-- Kinematics -->
             <wheel_separation>0.35</wheel_separation>
-            <wheel_diameter>0.1</wheel_diameter>
+            <wheel_diameter>0.066</wheel_diameter>
             <!-- Limits -->
             <max_linear_acceleration>10</max_linear_acceleration>
@@ -18,5 +18,5 @@
             <odom_publisher_frequency>30</odom_publisher_frequency>
             <topic>cmd_vel</topic>
-            <tf_topic>/tf</tf_topic>
+            <tf_topic>tf</tf_topic>
         </plugin>
         <!-- Joint state publisher -->

File: description/lidar.xacro (robot description, xacro)
@@ -9,5 +9,5 @@
         <visual>
             <geometry>
-                <cylinder radius="0.05" length="0.04"/>
+                <cylinder radius="0.015" length="0.035"/>
             </geometry>
             <material name="red"/>
@@ -15,8 +15,8 @@
         <collision>
             <geometry>
-                <cylinder radius="0.05" length="0.04"/>
+                <cylinder radius="0.015" length="0.035"/>
             </geometry>
         </collision>
-        <xacro:inertial_cylinder mass="0.1" length="0.04" radius="0.05">
+        <xacro:inertial_cylinder mass="0.045" length="0.035" radius="0.015">
             <origin xyz="0 0 0" rpy="0 0 0"/>
         </xacro:inertial_cylinder>
@@ -24,4 +24,7 @@
     <gazebo reference="laser_frame">
         <material>Gazebo/Red</material>
+        <!-- <plugin filename="gz-sim-sensors-system" name="gz::sim::systems::Sensors">
+            <render_engine>ogre2</render_engine>
+        </plugin> -->
         <sensor name="laser_frame" type="gpu_lidar">
             <pose> 0 0 0 0 0 0 </pose>
@@ -40,11 +43,8 @@
                 </scan>
                 <range>
-                    <min>0.3</min>
+                    <min>0.12</min>
                     <max>12</max>
                 </range>
             </lidar>
-            <plugin filename="gz-sim-sensors-system" name="gz::sim::systems::Sensors">
-                <render_engine>ogre2</render_engine>
-            </plugin>
         </sensor>
     </gazebo>

File: description/robot.urdf.xacro (robot description, xacro)
@@ -2,5 +2,5 @@
 <robot xmlns:xacro="http://www.ros.org/wiki/xacro"  name="differential_drive_robot">
     <xacro:include filename="robot_core.xacro" />
-    <!-- <xacro:arg name="use_ros2_control" default="false"/>
+    <xacro:arg name="use_ros2_control" default="false"/>
     <xacro:if value="$(arg use_ros2_control)">
         <xacro:include filename="ros2_control.xacro" />
@@ -8,6 +8,5 @@
     <xacro:unless value="$(arg use_ros2_control)">
         <xacro:include filename="gazebo_control.xacro" />
-    </xacro:unless> -->
-    <xacro:include filename="gazebo_control.xacro"/>
+    </xacro:unless>
     <xacro:include filename="lidar.xacro" />
     <xacro:include filename="camera.xacro" />

File: description/robot_core.xacro (robot description, xacro)
@@ -60,5 +60,5 @@
         <origin xyz="0 0.175 0" rpy="-${pi/2} 0 0"/>
         <axis xyz="0 0 1"/>
-        <limit effort="200" velocity="20"/>
+        <limit effort="200" velocity="10"/>
         <dynamics damping="1.0" friction="1.0"/>
     </joint>
@@ -66,5 +66,5 @@
         <visual>
             <geometry>
-                <cylinder radius="0.05" length="0.04"/>
+                <cylinder radius="0.033" length="0.027"/>
             </geometry>
             <material name="blue"/>
@@ -72,15 +72,15 @@
         <collision>
             <geometry>
-                <cylinder radius="0.05" length="0.04"/>
+                <cylinder radius="0.033" length="0.027"/>
             </geometry>
         </collision>
-        <xacro:inertial_cylinder mass="0.1" length="0.04" radius="0.05">
+        <xacro:inertial_cylinder mass="0.0385" length="0.027" radius="0.033">
             <origin xyz="0 0 0" rpy="0 0 0"/>
         </xacro:inertial_cylinder>
     </link>
     <gazebo reference="left_wheel">
+        <material>Gazebo/Blue</material>
         <mu1>0.2</mu1>
         <mu2>0.2</mu2>
-        <material>Gazebo/Blue</material>
     </gazebo>
     <!-- RIGHT WHEEL LINK -->
@@ -90,5 +90,5 @@
         <origin xyz="0 -0.175 0" rpy="${pi/2} 0 0"/>
         <axis xyz="0 0 -1"/>
-        <limit effort="200" velocity="20"/>
+        <limit effort="200" velocity="10"/>
         <dynamics damping="1.0" friction="1.0"/>
     </joint>
@@ -96,5 +96,5 @@
         <visual>
             <geometry>
-                <cylinder radius="0.05" length="0.04"/>
+                <cylinder radius="0.033" length="0.027"/>
             </geometry>
             <material name="blue"/>
@@ -102,15 +102,15 @@
         <collision>
             <geometry>
-                <cylinder radius="0.05" length="0.04"/>
+                <cylinder radius="0.033" length="0.027"/>
             </geometry>
         </collision>
-        <xacro:inertial_cylinder mass="0.1" length="0.04" radius="0.05">
+        <xacro:inertial_cylinder mass="0.0385" length="0.027" radius="0.033">
             <origin xyz="0 0 0" rpy="0 0 0"/>
         </xacro:inertial_cylinder>
     </link>
     <gazebo reference="right_wheel">
+        <material>Gazebo/Blue</material>
         <mu1>0.2</mu1>
         <mu2>0.2</mu2>
-        <material>Gazebo/Blue</material>
     </gazebo>
     <!-- CASTER WHEEL LINK -->
@@ -123,5 +123,5 @@
         <visual>
             <geometry>
-                <sphere radius="0.05"/>
+                <sphere radius="0.035"/>
             </geometry>
             <material name="black"/>
@@ -129,8 +129,8 @@
         <collision>
             <geometry>
-                <sphere radius="0.05"/>
+                <sphere radius="0.035"/>
             </geometry>
         </collision>
-        <xacro:inertial_sphere mass="0.1" radius="0.05">
+        <xacro:inertial_sphere mass="0.1" radius="0.035">
             <origin xyz="0 0 0" rpy="0 0 0"/>
         </xacro:inertial_sphere>

File: description/ros2_control.xacro (robot description, xacro)
@@ -23,5 +23,5 @@
     </ros2_control>
     <gazebo>
-        <plugin filename="libgazebo_ros2_control.so" name="gazebo_ros2_control">
+        <plugin filename="gz-sim-diff-drive-system" name="gazebo_ros2_control">
             <parameters>$(find vehicle_bot)/config/my_controllers.yaml</parameters>
         </plugin>

Commit message: updated body dimension for real robot

File: description/camera.xacro (robot description, xacro)
@@ -4,5 +4,5 @@
         <parent link="chassis"/>
         <child link="camera_link"/>
-        <origin xyz="0.305 0 0.08" rpy="0 0 0"/>
+        <origin xyz="0.225 0 0.041" rpy="0 0 0"/>
     </joint>
     <link name="camera_link">

File: description/depth_camera.xacro (robot description, xacro)
@@ -4,5 +4,5 @@
         <parent link="chassis"/>
         <child link="camera_link"/>
-        <origin xyz="0.305 0 0.08" rpy="0 0 0"/>
+        <origin xyz="0.225 0 0.04" rpy="0 0 0"/>
     </joint>
     <link name="camera_link">

File: description/gazebo_control.xacro (robot description, xacro)
@@ -8,5 +8,5 @@
             <right_joint>right_wheel_joint</right_joint>
             <!-- Kinematics -->
-            <wheel_separation>0.35</wheel_separation>
+            <wheel_separation>0.172</wheel_separation>
             <wheel_diameter>0.066</wheel_diameter>
             <!-- Limits -->

File: description/lidar.xacro (robot description, xacro)
@@ -4,5 +4,5 @@
         <parent link="chassis"/>
         <child link="laser_frame"/>
-        <origin xyz="0.1 0 0.175" rpy="0 0 0"/>
+        <origin xyz="0.11 0 0.0995" rpy="0 0 0"/>
     </joint>
     <link name="laser_frame">
@@ -24,7 +24,4 @@
     <gazebo reference="laser_frame">
         <material>Gazebo/Red</material>
-        <!-- <plugin filename="gz-sim-sensors-system" name="gz::sim::systems::Sensors">
-            <render_engine>ogre2</render_engine>
-        </plugin> -->
         <sensor name="laser_frame" type="gpu_lidar">
             <pose> 0 0 0 0 0 0 </pose>

File: description/robot_core.xacro (robot description, xacro)
@@ -23,5 +23,5 @@
         <parent link="base_footprint"/>
         <child link="base_link"/>
-        <origin xyz="0 0 0.05" rpy="0 0 0"/>
+        <origin xyz="0 0 0.008" rpy="0 0 0"/>
     </joint>
     <link name="base_link">
@@ -31,22 +31,22 @@
         <parent link="base_link"/>
         <child link="chassis"/>
-        <origin xyz="-0.1 0 0"/>
+        <origin xyz="-0.06 0 0"/>
     </joint>
     <link name="chassis">
         <visual>
-            <origin xyz="0.15 0 0.075"/>
+            <origin xyz="0.11 0 0.041"/>
             <geometry>
-                <box size="0.3 0.3 0.15"/>
+                <box size="0.22 0.156 0.082"/>
             </geometry>
             <material name="white"/>
         </visual>
         <collision>
-            <origin xyz="0.15 0 0.075"/>
+            <origin xyz="0.11 0 0.041"/>
             <geometry>
-                <box size="0.3 0.3 0.15"/>
+                <box size="0.22 0.156 0.082"/>
             </geometry>
         </collision>
-        <xacro:inertial_box mass="0.5" x="0.3" y="0.3" z="0.15">
-            <origin xyz="0.15 0 0.075" rpy="0 0 0"/>
+        <xacro:inertial_box mass="1.0" x="0.22" y="0.156" z="0.082">
+            <origin xyz="0.11 0 0.041" rpy="0 0 0"/>
         </xacro:inertial_box>
     </link>
@@ -58,5 +58,5 @@
         <parent link="base_link"/>
         <child link="left_wheel"/>
-        <origin xyz="0 0.175 0" rpy="-${pi/2} 0 0"/>
+        <origin xyz="0 0.093 0.025" rpy="-${pi/2} 0 0"/>
         <axis xyz="0 0 1"/>
         <limit effort="2000" velocity="30"/>
@@ -66,5 +66,5 @@
         <visual>
             <geometry>
-                <cylinder radius="0.033" length="0.027"/>
+                <cylinder radius="0.033" length="0.026"/>
             </geometry>
             <material name="blue"/>
@@ -72,8 +72,8 @@
         <collision>
             <geometry>
-                <cylinder radius="0.033" length="0.027"/>
+                <cylinder radius="0.033" length="0.026"/>
             </geometry>
         </collision>
-        <xacro:inertial_cylinder mass="0.0385" length="0.027" radius="0.033">
+        <xacro:inertial_cylinder mass="0.0385" length="0.026" radius="0.033">
             <origin xyz="0 0 0" rpy="0 0 0"/>
         </xacro:inertial_cylinder>
@@ -88,5 +88,5 @@
         <parent link="base_link"/>
         <child link="right_wheel"/>
-        <origin xyz="0 -0.175 0" rpy="${pi/2} 0 0"/>
+        <origin xyz="0 -0.093 0.025" rpy="${pi/2} 0 0"/>
         <axis xyz="0 0 -1"/>
         <limit effort="2000" velocity="30"/>
@@ -96,5 +96,5 @@
         <visual>
             <geometry>
-                <cylinder radius="0.033" length="0.027"/>
+                <cylinder radius="0.033" length="0.026"/>
             </geometry>
             <material name="blue"/>
@@ -102,8 +102,8 @@
         <collision>
             <geometry>
-                <cylinder radius="0.033" length="0.027"/>
+                <cylinder radius="0.033" length="0.026"/>
             </geometry>
         </collision>
-        <xacro:inertial_cylinder mass="0.0385" length="0.027" radius="0.033">
+        <xacro:inertial_cylinder mass="0.0385" length="0.026" radius="0.033">
             <origin xyz="0 0 0" rpy="0 0 0"/>
         </xacro:inertial_cylinder>
@@ -118,10 +118,10 @@
         <parent link="chassis"/>
         <child link="caster_wheel"/>
-        <origin xyz="0.24 0 0"/>
+        <origin xyz="0.17 0 0"/>
     </joint>
     <link name="caster_wheel">
         <visual>
             <geometry>
-                <sphere radius="0.035"/>
+                <sphere radius="0.008"/>
             </geometry>
             <material name="black"/>
@@ -129,8 +129,8 @@
         <collision>
             <geometry>
-                <sphere radius="0.035"/>
+                <sphere radius="0.008"/>
             </geometry>
         </collision>
-        <xacro:inertial_sphere mass="0.05" radius="0.035">
+        <xacro:inertial_sphere mass="0.02" radius="0.008">
             <origin xyz="0 0 0" rpy="0 0 0"/>
         </xacro:inertial_sphere>
