Commit message: updated gazebo contents commands etc

File: description/camera.xacro (robot description, xacro)
@@ -4,12 +4,20 @@
         <parent link="chassis"/>
         <child link="camera_link"/>
-        <origin xyz="0.225 0 0.041" rpy="0 0 0"/>
+        <origin xyz="0.192 0 0.097" rpy="0 0 0"/>
     </joint>
     <link name="camera_link">
-        <visual>
+        <pose>0 0 0 0 0 0</pose>
+        <collision name='collision'>
+            <origin xyz="0 0 0" rpy="0 0 0"/>
             <geometry>
-                <box size="0.01 0.03 0.03"/>
+                <box size="0.018 0.07 0.03"/>
             </geometry>
-            <material name="red"/>
+        </collision>
+        <visual name='camera_link_visual'>
+            <origin xyz="0 0 0" rpy="0 0 0"/>
+            <geometry>
+                <box size="0.018 0.07 0.03"/>
+            </geometry>
+            <material name="black"/>
         </visual>
     </link>
@@ -21,16 +29,16 @@
     <link name="camera_link_optical"></link>
     <gazebo reference="camera_link_optical">
-        <material>Gazebo/Red</material>
+        <material>Gazebo/Black</material>
         <!-- <plugin filename="gz-sim-sensors-system" name="gz::sim::systems::Sensors">
             <render_engine>ogre2</render_engine>
         </plugin> -->
-        <sensor name="camera_link_optical" type="camera">
+        <sensor name="camera" type="camera">
             <pose> 0 0 0 ${pi/2} ${-pi/2} 0 </pose>
-            <always_on>true</always_on>
+            <always_on>1</always_on>
             <visualize>true</visualize>
             <update_rate>10</update_rate>
             <topic>camera</topic>
-            <gz_frame_id>camera_link_optical</gz_frame_id>
-            <camera>
+            <optical_frame_id>camera_link_optical</optical_frame_id>
+            <camera name="logicool_c270n">
                 <camera_info_topic>camera/camera_info</camera_info_topic>
                 <horizontal_fov>1.089</horizontal_fov>  <!-- this unit is radians -->

File: description/gazebo_control.xacro (robot description, xacro)
@@ -9,5 +9,5 @@
             <!-- Kinematics -->
             <wheel_separation>0.172</wheel_separation>
-            <wheel_diameter>0.066</wheel_diameter>
+            <wheel_radius>0.033</wheel_radius>
             <!-- Limits -->
             <max_linear_acceleration>10</max_linear_acceleration>
@@ -16,10 +16,10 @@
             <min_linear_velocity>-30</min_linear_velocity> -->
             <!-- Input -->
-            <topic>cmd_vel</topic>
+            <topic>/cmd_vel</topic>
             <!-- Output -->
-            <odom_topic>odom</odom_topic>
             <frame_id>odom</frame_id>
             <child_frame_id>base_footprint</child_frame_id>
-            <odom_publish_frequency>5</odom_publish_frequency>
+            <odom_topic>odom</odom_topic>
+            <odom_publisher_frequency>5</odom_publisher_frequency>
             <tf_topic>tf</tf_topic>
         </plugin>

File: description/lidar.xacro (robot description, xacro)
@@ -4,19 +4,26 @@
         <parent link="chassis"/>
         <child link="laser_frame"/>
-        <origin xyz="0.11 0 0.0995" rpy="0 0 0"/>
+        <origin xyz="0.11 0 0.127" rpy="0 0 0"/>
     </joint>
     <link name="laser_frame">
         <visual>
             <geometry>
-                <cylinder radius="0.015" length="0.035"/>
+                <cylinder radius="0.015" length="0.013"/>
             </geometry>
             <material name="red"/>
         </visual>
+        <visual>
+            <origin xyz="0 0 -0.03"/>
+            <geometry>
+                <box size="0.035 0.035 0.047"/>
+            </geometry>
+            <material name="black"/>
+        </visual>
         <collision>
             <geometry>
-                <cylinder radius="0.015" length="0.035"/>
+                <cylinder radius="0.015" length="0.013"/>
             </geometry>
         </collision>
-        <xacro:inertial_cylinder mass="0.045" length="0.035" radius="0.015">
+        <xacro:inertial_cylinder mass="0.045" length="0.013" radius="0.015">
             <origin xyz="0 0 0" rpy="0 0 0"/>
         </xacro:inertial_cylinder>

File: description/robot_core.xacro (robot description, xacro)
@@ -35,5 +35,5 @@
     </material>
     <!-- BASE FOOTPRINT -->
-    <link name="base_footprint"/>
+    <link name="base_footprint"></link>
     <!-- BASE LINK -->
     <joint name="base_joint" type="fixed">
@@ -42,6 +42,5 @@
         <origin xyz="0 0 ${chassis_offset_z}" rpy="0 0 0"/>
     </joint>
-    <link name="base_link">
-    </link>
+    <link name="base_link"></link>
     <!-- CHASSIS LINK -->
     <joint name="chassis_joint" type="fixed">
